Commit message: Add files

File: urdf/turtlebot3_burger.gazebo.xacro (robot description, xacro)
@@ -96,4 +96,36 @@
     <sensor type="gpu_ray" name="lds_lfcd_sensor">
       <pose>0 0 0 0 0 0</pose>
+      <visualize>false</visualize>
+      <update_rate>5</update_rate>
+      <ray>
+        <scan>
+          <horizontal>
+            <samples>360</samples>
+            <resolution>1</resolution>
+            <min_angle>0</min_angle>
+            <max_angle>6.283</max_angle>
+          </horizontal>
+        </scan>
+        <range>
+          <min>0.120</min>
+          <max>10.0</max>
+          <resolution>0.015</resolution>
+        </range>
+        <noise>
+          <type>gaussian</type>
+          <mean>0.0</mean>
+          <stddev>0.01</stddev>
+        </noise>
+      </ray>
+      <plugin name="gazebo_ros_lds_lfcd_controller" filename="libgazebo_ros_gpu_laser.so">
+        <topicName>scan</topicName>
+        <frameName>base_scan</frameName>
+      </plugin>
+    </sensor>
+  </gazebo>
+  <gazebo reference="head_base_scan">
+    <material>Gazebo/FlatBlack</material>
+    <sensor type="gpu_ray" name="head_lds_lfcd_sensor">
+      <pose>0 0 0 0 0 0</pose>
       <visualize>$(arg laser_visual)</visualize>
       <update_rate>5</update_rate>
@@ -119,6 +151,6 @@
       </ray>
       <plugin name="gazebo_ros_lds_lfcd_controller" filename="libgazebo_ros_gpu_laser.so">
-        <topicName>scan</topicName>
-        <frameName>base_scan</frameName>
+        <topicName>head_scan</topicName>
+        <frameName>head_base_scan</frameName>
       </plugin>
     </sensor>

File: urdf/turtlebot3_burger.urdf.xacro (robot description, xacro)
@@ -116,6 +116,6 @@
     <parent link="base_link"/>
     <child link="base_scan"/>
-    <!-- <origin xyz="-0.032 0 0.172" rpy="0 0 0"/> -->
-    <origin xyz="-0.032 0 0.772" rpy="0 0 0"/>
+    <origin xyz="-0.032 0 0.172" rpy="0 0 0"/>
+    <!-- <origin xyz="-0.032 0 0.772" rpy="0 0 0"/> -->
   </joint>
   <link name="base_scan">
@@ -141,4 +141,32 @@
     </inertial>
   </link>
+  <joint name="head_scan_joint" type="fixed">
+    <parent link="base_link"/>
+    <child link="head_base_scan"/>
+    <!-- <origin xyz="-0.032 0 0.172" rpy="0 0 0"/> -->
+    <origin xyz="-0.032 0 0.772" rpy="0 0 0"/>
+  </joint>
+  <link name="head_base_scan">
+    <visual>
+      <origin xyz="0 0 0.0" rpy="0 0 0"/>
+      <geometry>
+        <mesh filename="package://turtlebot3_description/meshes/sensors/lds.stl" scale="0.001 0.001 0.001"/>
+      </geometry>
+      <material name="dark"/>
+    </visual>
+    <!-- <collision>
+      <origin xyz="0.015 0 -0.0065" rpy="0 0 0"/>
+      <geometry>
+        <cylinder length="0.0315" radius="0.055"/>
+      </geometry>
+    </collision>
+    <inertial>
+      <mass value="0.114" />
+      <origin xyz="0 0 0" />
+      <inertia ixx="0.001" ixy="0.0" ixz="0.0"
+               iyy="0.001" iyz="0.0"
+               izz="0.001" />
+    </inertial> -->
+  </link>
   <joint name="camera_rgb_joint" type="fixed">
     <parent link="base_link"/>
